Commit message: 规划改成"最近 IK 关节目标"的工业做法, 并集成 WHEELTEC 柔性机械爪
问题一: 同一个位姿对应多组关节解(肘上/肘下、手腕翻转、J1/J4/J6 绕 ±360°),
OMPL 采样到哪组是随机的 —— "J1 转几度就够"的动作经常变成整条手臂绕大圈;
而默认的 KDL 插件是牛顿迭代, 本臂 J5 接近 ±90°(手腕奇异)时从种子不收敛就
改用随机种子重启, 于是同一个目标反复求解会落到不同分支上, 表现为"抓取动作
有时走最优轨迹、有时绕大圈"。

一、运动规划
- `kinematics.yaml`: KDL → `lma_kinematics_plugin/LMAKinematicsPlugin`,
  求解超时 5ms → 50ms。LMA 是阻尼最小二乘, 从种子出发几乎总能收敛到
  "离种子最近"的那一支(实测同目标同种子连续 10 次完全一致)
- `backend.py` 改成逐级回退的工业做法: **最近 IK 关节目标**(JointConstraint)
  → Pilz `PTP` → OMPL → 放宽容差的关节目标 → 位姿目标; 并记录轨迹的单关节最大
  行程, 超过 40° 就告警 —— 绕大圈从"看起来怪"变成可量化的数字
- `arena.transfer_tcp_z()`: 转场高度按"障碍顶面 + 间隙 + 工件挂深"显式算出来,
  不再复用预抓取悬停高度。抬不够时关节空间直线会撞, 规划器退回 OMPL 就绕出
  往外甩、往上拱的大弧(实测末端拱到 354mm、半径甩出 420mm 作业带)
- 修 `arena.py` 里"工件离支撑面 1mm"的两处漏算(reach_rows / source_area_top_z),
  提取成 `OBJECT_LIFT`, `scene_generator` 共用 —— 之前 arena_check 的"末端几何"
  与"末端可达性"会打印出互相差 1mm 的两套数字
- `arena_check` 新增"末端可达性"逐点校核(6 个工位的抓取/预抓取 + 料盒转场/投放);
  `docs/真机部署.md` 同步说明自检跑的就是这条链路

二、末端: WHEELTEC MS42DC 二指柔性爪(`gripper.STEP` + 厂商资料)
- 新增 `jaka_ros2/src/wheeltec_gripper/`: STEP→STL 转换脚本(可重跑)、实测几何
  (`config/gripper.yaml`)、装在 `dummy_tcp` 上的 URDF 宏、Gazebo 资源导出。
  STEP 不能直接用: Gazebo/MoveIt 只认三角网格, 而且 STEP 里没有"哪块是底座、
  哪块是手指"的语义, 两片指必须拆成两个转动关节才能张合
- 新增 `step_motor`(厂商串口驱动, 话题 `/motor_control`)、`serial_ros2`(依赖库);
  厂商原始资料(手册/固件/上位机/三维模型)进 `WHEELTEC 柔性机械爪/`
- 一个 `JAKA_GRIPPER=1` 同时切三处(URDF 模型 / 抓取高度 / 夹爪控制器), 拆开改
  就会出现"URDF 有夹爪、高度按法兰算"这种把手指戳进台面的组合; 默认仍是
  `none` —— 规则书要求的是行程 0–30mm 的电动平行夹爪
- 仿真 `SimGripper` 按工件宽度算指间角度走 `/gripper_controller/commands`,
  真机 `WheeltecGripper` 走 `/motor_control`(堵转自停, 所以"发一个够大的角度"
  就是"夹紧")

⚠ 可达性: 204.6mm 的指尖把抓取高度从 100.0 抬到 213.6mm, 而 580mm 臂展在
r=385mm 处工具朝下最多到 195.9mm —— 工位 4/6 抓不到, 料盒中心转场
(272.6 > 240.3)也抬不到。这不是参数没调好, 是臂展与爪长的几何结果, 真机同样
够不到; 数字、逐点校核与四个可选方案见 `docs/WHEELTEC柔性机械爪.md` 第 4 节。

实测: 默认(不装夹爪)赛道一 6/6 = 100.0 分(48.9s)、赛道二 12/12 = 150.0 分
(108.6s); `JAKA_GRIPPER=1` 跑一轮与可达性表逐点吻合 —— 工位 1/2/3/5 都抓到了
工件, 但抬去料盒全部规划失败, 4/6 连预抓取都到不了。Gazebo 里夹爪网格与碰撞体
正常加载(需要 `package.xml` 导出 `gazebo_model_path`, 否则夹爪隐形且没有碰撞)。

File: jaka_ros2/src/jaka_minicobo_moveit_config/config/jaka_minicobo.ros2_control.xacro (robot description, xacro)
@@ -1,5 +1,5 @@
 <?xml version="1.0"?>
 <robot xmlns:xacro="http://www.ros.org/wiki/xacro">
-    <xacro:macro name="jaka_minicobo_ros2_control" params="name initial_positions_file use_gazebo use_rviz_sim">
+    <xacro:macro name="jaka_minicobo_ros2_control" params="name initial_positions_file use_gazebo use_rviz_sim with_gripper">
         <xacro:property name="initial_positions" value="${xacro.load_yaml(initial_positions_file)['initial_positions']}"/>
         <ros2_control name="${name}" type="system">
@@ -57,4 +57,21 @@
                 <state_interface name="velocity"/>
             </joint>
+            <!-- 夹爪两片指: 由 gripper_controller 驱动(位置控制), 初始 0 = 张开 -->
+            <xacro:if value="${with_gripper}">
+              <joint name="gripper_jaw_l_joint">
+                  <command_interface name="position"/>
+                  <state_interface name="position">
+                    <param name="initial_value">0.0</param>
+                  </state_interface>
+                  <state_interface name="velocity"/>
+              </joint>
+              <joint name="gripper_jaw_r_joint">
+                  <command_interface name="position"/>
+                  <state_interface name="position">
+                    <param name="initial_value">0.0</param>
+                  </state_interface>
+                  <state_interface name="velocity"/>
+              </joint>
+            </xacro:if>
         </ros2_control>
     </xacro:macro>

File: jaka_ros2/src/jaka_minicobo_moveit_config/config/jaka_minicobo.urdf.xacro (robot description, xacro)
@@ -4,9 +4,22 @@
     <xacro:arg name="use_gazebo" default="false"/>
     <xacro:arg name="use_rviz_sim" default="false"/>
+    <!-- 末端夹爪: 默认**不装**(比赛规则书要求的是行程 0-30mm 的电动平行夹爪,
+         和裸法兰差不多长)。要挂 WHEELTEC MS42DC 二指柔性机械爪时(见
+         wheeltec_gripper 包), 设环境变量 JAKA_GRIPPER=1 —— arena.yaml 里的
+         tool.gripper 读的是同一个变量(jaka_competition_kit/arena.py), 所以
+         抓取高度会和 URDF 一起切过去, 不会出现"URDF 有夹爪、高度按法兰算"
+         这种把手指戳进台面的组合。
+         也可以显式传: xacro ... with_gripper:=true -->
+    <xacro:arg name="with_gripper" default="$(optenv JAKA_GRIPPER 0)"/>
     <!-- Import jaka_minicobo urdf file -->
     <xacro:include filename="$(find jaka_description)/urdf/jaka_minicobo.urdf" />
+    <!-- 末端夹爪(装在 dummy_tcp 上) -->
+    <xacro:include filename="$(find wheeltec_gripper)/urdf/wheeltec_gripper.urdf.xacro" />
+    <xacro:if value="$(arg with_gripper)">
+        <xacro:wheeltec_gripper prefix="" parent="dummy_tcp"/>
+    </xacro:if>
     <!-- Import control_xacro -->
     <xacro:include filename="jaka_minicobo.ros2_control.xacro" />
     <!-- <xacro:jaka_minicobo_ros2_control name="FakeSystem" initial_positions_file="$(arg initial_positions_file)"/> -->
-    <xacro:jaka_minicobo_ros2_control name="jaka_minicobo_hardware" initial_positions_file="$(arg initial_positions_file)" use_gazebo="$(arg use_gazebo)" use_rviz_sim="$(arg use_rviz_sim)" />
+    <xacro:jaka_minicobo_ros2_control name="jaka_minicobo_hardware" initial_positions_file="$(arg initial_positions_file)" use_gazebo="$(arg use_gazebo)" use_rviz_sim="$(arg use_rviz_sim)" with_gripper="$(arg with_gripper)" />
 </robot>
